File: STDC14-Adapter.kicad_pcb (KiCad board)
At the start: 2 copper layers, 22.9 x 30.5 mm, 3 parts, among them J1 Conn_ST_STDC14, J2 Conn_01x06, J3 Conn_01x06

Commit message: update pcb and add production files
Changed lines of the file:
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@@
 	(title_block
 		(title "STDC14 Adapter")
-		(date "2024-03-16")
+		(date "2024-03-31")
 		(rev "1.0")
-		(company "AM163")
-		(comment 4 "AISLER Project ID: LIZLXAFS")
+		(company "antoine163")
 	)
 	(layers
@@
 			(unlocked yes)
 			(layer "F.SilkS")
+			(hide yes)
 			(effects
 				(font
@@
 			(at 0 15.03 180)
 			(layer "F.Fab")
+			(hide yes)
 			(effects
 				(font
@@
 			(unlocked yes)
 			(layer "F.SilkS")
+			(hide yes)
 			(effects
 				(font
@@
 			(at 0 15.03 0)
 			(layer "F.Fab")
+			(hide yes)
 			(effects
 				(font
@@
 			(unlocked yes)
 			(layer "F.SilkS")
+			(hide yes)
 			(effects
 				(font
@@
 		)
 		(property "Value" "Conn_ST_STDC14"
-			(at 0 5.505 -90)
-			(layer "F.Fab")
+			(at 0 5.505 270)
+			(layer "F.Fab")
+			(hide yes)
 			(effects
 				(font
@@
 		)
 	)
-	(gr_text "RX"
+	(gr_text "TX"
 		(at 160.02 78.74 0)
 		(layer "F.SilkS")
@@
 		)
 	)
-	(gr_text "TX"
+	(gr_text "RX"
 		(at 160.02 81.28 0)
 		(layer "F.SilkS")
