File: STDC14-Adapter.kicad_sch (KiCad schematic)
At the start: 3 parts, among them J1 Conn_ST_STDC14, J2 Conn_01x06, J3 Conn_01x06

Commit message: update pcb and add production files
Other:
- company: AM163 -> antoine163
Changed lines of the file:
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@@
 	(title_block
 		(title "STDC14 Adapter")
-		(date "2024-03-16")
+		(date "2024-03-31")
 		(rev "1.0")
-		(company "AM163")
+		(company "antoine163")
 	)
 	(junction
